File: CircuitDesign/arenaPCBv1/_autosave-arenaPCBv1.kicad_sch (KiCad schematic)
At the start: 25 parts, among them Q1 IRLB3034

Commit message: Before redoing PCB
Parts:
- C3, C6: footprint Capacitor_SMD:CP_Elec_6.3x5.2 -> Capacitor_SMD:CP_Elec_6.3x4.5
Changed lines of the file:
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@@
       (effects (font (size 1.27 1.27)) (justify left))
     )
-    (property "Footprint" "Capacitor_SMD:CP_Elec_6.3x5.2" (at 135.89 128.27 0)
+    (property "Footprint" "Capacitor_SMD:CP_Elec_6.3x4.5" (at 135.89 128.27 0)
       (effects (font (size 1.27 1.27)) hide)
     )
@@
       (effects (font (size 1.27 1.27)) (justify left))
     )
-    (property "Footprint" "Capacitor_SMD:CP_Elec_6.3x5.2" (at 135.89 105.41 0)
+    (property "Footprint" "Capacitor_SMD:CP_Elec_6.3x4.5" (at 135.89 105.41 0)
       (effects (font (size 1.27 1.27)) hide)
     )
