File: CircuitDesign/arenaPCBv2/arenaPCBv2.kicad_sch (KiCad schematic)
At the start: 26 parts, among them Q1 IRLB3034

Commit message: pcb updates and other stuff
Parts:
- removed J10: ~, symbol 1_Bachelors_Symbols:SINGLE_PIN
- added J10: ~, symbol 1_bachelor_symbols:MISC_Connector
- J5: symbol 1_Bachelors_Symbols:LED_Connector -> 1_bachelor_symbols:LED_Connector
Connections:
- net GND: now also J10.2 (Pin_2)
- net at J9.18 (MISC): now also J10.1 (pin_1)

Commit message: SMD PCB done
Parts:
- removed J10: ~, symbol 1_bachelor_symbols:MISC_Connector
- D1, D2: footprint 2_Bachelors_footprints:S12GCH -> 2_bachelors_footprints:S12GCH
- F1: value MF-RG650-0 -> 2920L600/12MR; footprint Fuse:Fuse_Bourns_MF-RG650 -> Fuse:Fuse_2920_7451Metric_Pad2.10x5.45mm_HandSolder
- J1: footprint 2_Bachelors_footprints:conn2_1-1123723-2_TEC -> 2_bachelors_footprints:CONN_MTA_100_2
- J2, J4: footprint 2_Bachelors_footprints:CONN_B4B-ZRLFSN_JST -> 2_bachelors_footprints:B4B-ZR-SM4-TFT
- J3: footprint 2_Bachelors_footprints:CONN_B2B-ZRLFSN_JST -> 2_bachelors_footprints:B2B-ZR-SM4-TFT
- J5: footprint Connector_PinSocket_2.54mm:PinSocket_1x02_P2.54mm_Vertical -> 2_bachelors_footprints:led_header_p2.54_2pin
- J6: footprint 2_Bachelors_footprints:LP127 -> 2_bachelors_footprints:TERMINAL_BLOCK_5081
- J7: footprint 2_Bachelors_footprints:CONN_B4P-VH_JST -> 2_bachelors_footprints:CONN_MTA_100_4
- J8: footprint 2_Bachelors_footprints:CONN_B6B_VH_JST -> 2_bachelors_footprints:CONN_MTA_100_6
- J9: footprint Connector_JST:JST_PHD_B16B-PHDSS_2x08_P2.00mm_Vertical -> 2_bachelors_footprints:CONN_MOLEX_18p_2.00mm; symbol 1_Bachelors_Symbols:PH{colon}2.54MM 2*6P -> 1_bachelor_symbols:PH{colon}2.54MM 2*6P
- Q1: value IRLB3034 -> BSC007N04LS6; footprint 2_Bachelors_footprints:IRF520N -> 2_bachelors_footprints:PG-TDSON-8-6_INF
- U1, U2: footprint Module:Pololu_Breakout-16_15.2x20.3mm -> 2_bachelors_footprints:CONN_BREAKOUT_BOARDS
Connections:
- net SDA: now also J9.18 (SDA); no longer J9.15 (SDA)
- no-connect marks 6 -> 7
Changed lines of the file:
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@@
   (junction (at 90.17 25.4) (diameter 0) (color 0 0 0 0)
-  )
-  (junction (at 182.88 95.25) (diameter 0) (color 0 0 0 0)
   )
   (junction (at 95.25 48.26) (diameter 0) (color 0 0 0 0)
@@
   (no_connect (at 90.17 119.38))
   (no_connect (at 121.92 119.38))
+  (no_connect (at 130.81 83.82))
   (no_connect (at 121.92 123.19))
   (no_connect (at 90.17 123.19))
@@
     (stroke (width 0) (type default))
   )
-  (wire (pts (xy 167.64 95.25) (xy 182.88 95.25))
-    (stroke (width 0) (type default))
-  )
   (wire (pts (xy 31.75 25.4) (xy 44.45 25.4))
     (stroke (width 0) (type default))
@@
     (stroke (width 0) (type default))
   )
-  (wire (pts (xy 125.73 96.52) (xy 153.67 96.52))
-    (stroke (width 0) (type default))
-  )
   (wire (pts (xy 217.17 21.59) (xy 217.17 22.86))
     (stroke (width 0) (type default))
@@
     (stroke (width 0) (type default))
   )
-  (wire (pts (xy 167.64 91.44) (xy 167.64 95.25))
-    (stroke (width 0) (type default))
-  )
   (wire (pts (xy 91.44 36.83) (xy 85.09 36.83))
     (stroke (width 0) (type default))
@@
     (stroke (width 0) (type default))
   )
-  (wire (pts (xy 153.67 96.52) (xy 153.67 138.43))
+  (wire (pts (xy 153.67 86.36) (xy 153.67 138.43))
     (stroke (width 0) (type default))
   )
@@
     (stroke (width 0) (type default))
   )
-  (wire (pts (xy 161.29 86.36) (xy 161.29 88.9))
-    (stroke (width 0) (type default))
-  )
   (wire (pts (xy 95.25 25.4) (xy 90.17 25.4))
     (stroke (width 0) (type default))
@@
     (stroke (width 0) (type default))
   )
-  (wire (pts (xy 125.73 83.82) (xy 130.81 83.82))
-    (stroke (width 0) (type default))
-  )
   (wire (pts (xy 170.18 127) (xy 170.18 125.73))
     (stroke (width 0) (type default))
@@
     (stroke (width 0) (type default))
   )
-  (wire (pts (xy 153.67 86.36) (xy 161.29 86.36))
-    (stroke (width 0) (type default))
-  )
   (wire (pts (xy 67.31 83.82) (xy 67.31 85.09))
     (stroke (width 0) (type default))
@@
   )
   (wire (pts (xy 111.76 59.69) (xy 111.76 71.12))
-    (stroke (width 0) (type default))
-  )
-  (wire (pts (xy 161.29 88.9) (xy 167.64 88.9))
-    (stroke (width 0) (type default))
-  )
-  (wire (pts (xy 125.73 83.82) (xy 125.73 96.52))
     (stroke (width 0) (type default))
   )
@@
       (effects (font (size 1.27 1.27)))
     )
-    (property "Footprint" "2_Bachelors_footprints:LP127" (at 31.75 78.74 0)
+    (property "Footprint" "2_bachelors_footprints:TERMINAL_BLOCK_5081" (at 31.75 78.74 0)
       (effects (font (size 1.27 1.27)) hide)
     )
@@
       (effects (font (size 1.27 1.27)) (justify left))
     )
-    (property "Value" "IRLB3034" (at 194.31 31.75 0)
-      (effects (font (size 1.27 1.27)) (justify left))
-    )
-    (property "Footprint" "2_Bachelors_footprints:IRF520N" (at 194.31 32.385 0)
+    (property "Value" "BSC007N04LS6" (at 194.31 31.75 0)
+      (effects (font (size 1.27 1.27)) (justify left))
+    )
+    (property "Footprint" "2_bachelors_footprints:PG-TDSON-8-6_INF" (at 194.31 32.385 0)
       (effects (font (size 1.27 1.27) italic) (justify left) hide)
     )
@@
       (effects (font (size 1.27 1.27)))
     )
-    (property "Footprint" "2_Bachelors_footprints:CONN_B4B-ZRLFSN_JST" (at 190.5 151.13 0)
+    (property "Footprint" "2_bachelors_footprints:B4B-ZR-SM4-TFT" (at 190.5 151.13 0)
       (effects (font (size 1.27 1.27)) hide)
     )
@@
       (effects (font (size 1.27 1.27)) (justify left))
     )
-    (property "Footprint" "2_Bachelors_footprints:S12GCH" (at 207.01 27.94 0)
+    (property "Footprint" "2_bachelors_footprints:S12GCH" (at 207.01 27.94 0)
       (effects (font (size 1.27 1.27)) hide)
     )
@@
       (effects (font (size 1.27 1.27)))
     )
-    (property "Footprint" "2_Bachelors_footprints:CONN_B6B_VH_JST" (at 204.47 100.33 0)
+    (property "Footprint" "2_bachelors_footprints:CONN_MTA_100_6" (at 204.47 100.33 0)
       (effects (font (size 1.27 1.27)) hide)
     )
@@
       (effects (font (size 1.27 1.27)))
     )
-    (property "Footprint" "2_Bachelors_footprints:CONN_B4B-ZRLFSN_JST" (at 209.55 151.13 0)
+    (property "Footprint" "2_bachelors_footprints:B4B-ZR-SM4-TFT" (at 209.55 151.13 0)
       (effects (font (size 1.27 1.27)) hide)
     )
@@
       (effects (font (size 1.27 1.27)) (justify left))
     )
-    (property "Footprint" "2_Bachelors_footprints:S12GCH" (at 55.88 81.28 0)
+    (property "Footprint" "2_bachelors_footprints:S12GCH" (at 55.88 81.28 0)
       (effects (font (size 1.27 1.27)) hide)
     )
@@
       (effects (font (size 1.27 1.27)))
     )
-    (property "Footprint" "2_Bachelors_footprints:CONN_B2B-ZRLFSN_JST" (at 209.55 55.88 0)
+    (property "Footprint" "2_bachelors_footprints:B2B-ZR-SM4-TFT" (at 209.55 55.88 0)
       (effects (font (size 1.27 1.27)) hide)
     )
@@
       (effects (font (size 1.27 1.27)))
     )
-    (property "Footprint" "Module:Pololu_Breakout-16_15.2x20.3mm" (at 105.41 115.57 0)
+    (property "Footprint" "2_bachelors_footprints:CONN_BREAKOUT_BOARDS" (at 105.41 115.57 0)
       (effects (font (size 1.27 1.27)) hide)
     )
@@
       (effects (font (size 1.27 1.27)))
     )
-    (property "Footprint" "2_Bachelors_footprints:conn2_1-1123723-2_TEC" (at 226.06 20.32 0)
+    (property "Footprint" "2_bachelors_footprints:CONN_MTA_100_2" (at 226.06 20.32 0)
       (effects (font (size 1.27 1.27)) hide)
     )
@@
     )
   )
-  (symbol (lib_id "1_bachelor_symbols:MISC_Connector") (at 175.26 90.17 0) (unit 1)
-    (in_bom yes) (on_board yes) (dnp no)
-    (property "Reference" "J10" (at 173.99 82.55 0)
-      (effects (font (size 1.27 1.27)) (justify left))
-    )
-    (property "Value" "~" (at 173.99 86.36 0)
-      (effects (font (size 1.27 1.27)))
-    )
-    (property "Footprint" "" (at 173.99 86.36 0)
-      (effects (font (size 1.27 1.27)) hide)
-    )
-    (property "Datasheet" "" (at 173.99 86.36 0)
-      (effects (font (size 1.27 1.27)) hide)
-    )
-    (pin "1")
-    (pin "2")
-    (instances
-      (project "arenaPCBv2"
-        (path "/aeb80c4e-8a5b-46ea-8e16-d30fa5558bce"
-          (reference "J10") (unit 1)
-        )
-      )
-    )
-  )
   (symbol (lib_id "1_Bachelors_Symbols:DRV8825_Stepper_Motor_Driver_Carrier") (at 64.77 34.29 0) (unit 1)
     (in_bom yes) (on_board yes) (dnp no)
@@
       (effects (font (size 1.27 1.27)))
     )
-    (property "Footprint" "Module:Pololu_Breakout-16_15.2x20.3mm" (at 64.77 13.97 0)
+    (property "Footprint" "2_bachelors_footprints:CONN_BREAKOUT_BOARDS" (at 64.77 13.97 0)
       (effects (font (size 1.27 1.27)) hide)
     )
@@
       (effects (font (size 1.27 1.27)))
     )
-    (property "Footprint" "2_Bachelors_footprints:CONN_B4P-VH_JST" (at 92.71 34.29 0)
+    (property "Footprint" "2_bachelors_footprints:CONN_MTA_100_4" (at 92.71 34.29 0)
       (effects (font (size 1.27 1.27)) hide)
     )
@@
       (effects (font (size 1.27 1.27)))
     )
-    (property "Value" "MF-RG650-0\n" (at 45.72 74.93 90)
-      (effects (font (size 1.27 1.27)))
-    )
-    (property "Footprint" "Fuse:Fuse_Bourns_MF-RG650" (at 45.72 79.248 90)
+    (property "Value" "2920L600/12MR\n" (at 45.72 74.93 90)
+      (effects (font (size 1.27 1.27)))
+    )
+    (property "Footprint" "Fuse:Fuse_2920_7451Metric_Pad2.10x5.45mm_HandSolder" (at 45.72 79.248 90)
       (effects (font (size 1.27 1.27)) hide)
     )
@@
       (effects (font (size 1.27 1.27)))
     )
-    (property "Footprint" "Connector_PinSocket_2.54mm:PinSocket_1x02_P2.54mm_Vertical" (at 99.06 77.47 0)
+    (property "Footprint" "2_bachelors_footprints:led_header_p2.54_2pin" (at 99.06 77.47 0)
       (effects (font (size 1.27 1.27)) hide)
     )
@@
     )
   )
-  (symbol (lib_id "1_Bachelors_Symbols:PH{colon}2.54MM 2*6P") (at 142.24 72.39 0) (unit 1)
+  (symbol (lib_id "1_bachelor_symbols:PH{colon}2.54MM 2*6P") (at 142.24 72.39 0) (unit 1)
     (in_bom yes) (on_board yes) (dnp no)
     (property "Reference" "J9" (at 142.24 59.69 0)
@@
       (effects (font (size 1.27 1.27)))
     )
-    (property "Footprint" "Connector_JST:JST_PHD_B16B-PHDSS_2x08_P2.00mm_Vertical" (at 123.19 72.39 0)
-      (effects (font (size 1.27 1.27)) hide)
-    )
+    (property "Footprint" "2_bachelors_footprints:CONN_MOLEX_18p_2.00mm" (at 123.19 72.39 0)
+      (effects (font (size 1.27 1.27)) hide)
+    )
